File: moleblink/moleblink.kicad_pcb (KiCad board)
At the start: 2 copper layers, 40.6 x 48.5 mm, 31 parts, among them Q1 IRFML8244, SW1 JS202011JCQN, SW2 PTS526 SK15 SMTR2 LFS, U1 ATtiny85V-10SU, U2 74HC595

Commit message: Update moleblink.kicad_pcb
Parts:
- removed the G*** at (142.4, 114.6)
- added G***: LOGO, crest:blacker_mask, F.Cu at (142.2, 113.8)
Other:
- board text added: "MoleBlink"
- board text removed: "RuddBlink"
